Commit message: 过渡阶段1.0

File: models/ninezzhou/urdf/ninezzhou.urdf (robot description, URDF)
Before this commit: robot ninezzhou, 10 links, 9 joints
Links:
- added link tool0
Joints:
- added joint tool0_fixed: type fixed, parent Link9, child tool0, origin xyz=0.235 0 0 rpy=0 0 0

Commit message: fix(motion): 修正J1模型坐标与反馈保护
增加九轴标定姿态表和离线逐组采集，记录验证结果与现场缺口

File: models/ninezzhou/urdf/ninezzhou.urdf (robot description, URDF)
Before this commit: robot ninezzhou, 11 links, 10 joints
Joints:
- joint J1: limit lower=0 upper=0.585 effort=1000 velocity=0.2 -> lower=0 upper=0.5 effort=1000 velocity=0.2; origin xyz=0 0 0 rpy=0 0 0 -> xyz=0 0 0.085 rpy=0 0 0

File: models/ninezzhou/urdf/ninezzhou_collision.urdf (robot description, URDF)
Before this commit: robot ninezzhou, 11 links, 10 joints
Joints:
- joint J1: limit lower=0 upper=0.585 effort=1000 velocity=0.2 -> lower=0 upper=0.5 effort=1000 velocity=0.2; origin xyz=0 0 0 rpy=0 0 0 -> xyz=0 0 0.085 rpy=0 0 0
